Commit message: I successfully added a shape to the visualization. Read the Visualization_Readme for a detailed description, in the raven_visualization folder. I also did an optimization for the visualization itself - the motor models are large files, so I replaced them with simple boxes to ease the suffering of the computer. It's mostly a function of Oracle VirtualBox's seeming unwillingness to use all 4GB of my graphics memory, though, and the optimization only gave a boost of 1-3 FPS besides. I'd be willing to work on that some more. All of this only took about 2 days - the rest of my time was spent learning how ROS worked and such. Very educational!

File: raven_visualization/ravenII_2arm.urdf (robot description, URDF)
Before this commit: robot raven_2, 17 links, 16 joints
Links:
- added link box_link; visual box size=0.1 0.1 0.1
- link 0_link: geometry visual box size=0.001 0.001 0.001
- link base_link_L: geometry visual box size=0.43 0.25 0.32
- link base_link_R: geometry visual box size=0.43 0.25 0.32
Joints:
- added joint box_joint: type fixed, parent 0_link, child box_link, origin xyz=0.0 0.00 0 rpy=0 0 0, limit lower=0.0 upper=3.1415 effort=1000.0 velocity=0.5

Commit message: Switched to urdf for the Gazebo visualization. That should work now.

File: raven_visualization/ravenII_2arm.urdf (robot description, URDF)
Before this commit: robot raven_2, 18 links, 17 joints
Links:
- link 0_link: mass None -> 1; geometry collision box size=0.01 0.01 0.01; visual box size=0.01 0.01 0.01
- link base_link_L: mass None -> 1
- link base_link_R: mass None -> 1
- link box_link: mass None -> 1; geometry visual box size=0.01 0.01 0.01
- link grasper1_L: mass None -> 1
- link grasper1_R: mass None -> 1
- link grasper2_L: mass None -> 1
- link grasper2_R: mass None -> 1
- link instrument_shaft_L: mass None -> 1
- link instrument_shaft_R: mass None -> 1
- link link1_L: mass None -> 1
- link link1_R: mass None -> 1
- link link2_L: mass None -> 1
- link link2_R: mass None -> 1
- link link3_L: mass None -> 1
- link link3_R: mass None -> 1
- link wrist_L: mass None -> 1
- link wrist_R: mass None -> 1

Commit message: Made the arms affected by Gazebo's physics engine. They're rooted to the world plane by a single fixed joint. Still need to add collision meshes to the rest of the links, at some point. Should be pretty easy, so I wouldn't worry too much about it now.

File: raven_visualization/ravenII_2arm.urdf (robot description, URDF)
Before this commit: robot raven_2, 18 links, 17 joints
Links:
- added link world
Joints:
- added joint fixed: type fixed, parent world, child 0_link

Commit message: Added collision tags to Raven arms, a simple sphere that you can nudge into the arms in the way specified by the Box journal entry.

File: raven_visualization/ravenII_2arm.urdf (robot description, URDF)
Before this commit: robot raven_2, 19 links, 18 joints
Links:
- link base_link_R: geometry collision box size=0.43 0.25 0.32; visual box size=0.43 0.25 0.32
- link box_link: geometry collision box size=0.01 0.01 0.01; visual box size=0.01 0.01 0.01
- link grasper1_L: geometry collision mesh filename=package://raven_visualization/Raven_files/left_arm/grasper_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; visual mesh filename=package://raven_visualization/Raven_files/left_arm/grasper_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
- link grasper1_R: geometry collision mesh filename=package://raven_visualization/Raven_files/right_arm/grasper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; visual mesh filename=package://raven_visualization/Raven_files/right_arm/grasper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
- link grasper2_L: geometry collision mesh filename=package://raven_visualization/Raven_files/left_arm/grasper_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; visual mesh filename=package://raven_visualization/Raven_files/left_arm/grasper_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
- link grasper2_R: geometry collision mesh filename=package://raven_visualization/Raven_files/right_arm/grasper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; visual mesh filename=package://raven_visualization/Raven_files/right_arm/grasper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
- link instrument_shaft_L: geometry collision mesh filename=package://raven_visualization/Raven_files/left_arm/instrume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; visual mesh filename=package://raven_visualization/Raven_files/left_arm/instrume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
- link instrument_shaft_R: geometry collision mesh filename=package://raven_visualization/Raven_files/right_arm/instrum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; visual mesh filename=package://raven_visualization/Raven_files/right_arm/instrum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
- link link1_L: geometry collision mesh filename=package://raven_visualization/Raven_files/left_arm/link1_w_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; visual mesh filename=package://raven_visualization/Raven_files/left_arm/link1_w_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
- link link1_R: geometry collision mesh filename=package://raven_visualization/Raven_files/right_arm/link1_w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; visual mesh filename=package://raven_visualization/Raven_files/right_arm/link1_w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
- link link2_L: geometry collision mesh filename=package://raven_visualization/Raven_files/left_arm/link2.dae; visual mesh filename=package://raven_visualization/Raven_files/left_arm/link2.dae
- link link2_R: geometry collision mesh filename=package://raven_visualization/Raven_files/right_arm/link2.d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; visual mesh filename=package://raven_visualization/Raven_files/right_arm/link2.d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
- link link3_L: geometry collision mesh filename=package://raven_visualization/Raven_files/left_arm/link3.dae; visual mesh filename=package://raven_visualization/Raven_files/left_arm/link3.dae
- link link3_R: geometry collision mesh filename=package://raven_visualization/Raven_files/right_arm/link3.d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; visual mesh filename=package://raven_visualization/Raven_files/right_arm/link3.d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
- link wrist_L: geometry collision mesh filename=package://raven_visualization/Raven_files/left_arm/wrist.dae; visual mesh filename=package://raven_visualization/Raven_files/left_arm/wrist.dae
- link wrist_R: geometry collision mesh filename=package://raven_visualization/Raven_files/right_arm/wrist.d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; visual mesh filename=package://raven_visualization/Raven_files/right_arm/wrist.d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

Commit message: Added joint state publisher gui to the launch file, so that you can control the joints in real-time. Don't ask me why I didn't think of this sooner, because I have no earthly idea.

File: raven_visualization/ravenII_2arm.urdf (robot description, URDF)
Before this commit: robot raven_2, 19 links, 18 joints
Links:
- removed link box_link
- link 0_link: geometry collision box size=0.01 0.01 0.01; visual box size=0.001 0.001 0.001
Joints:
- removed joint box_joint

Commit message: This one, I'm sure of it. This is it!

File: raven_visualization/ravenII_2arm.urdf (robot description, URDF)
Before this commit: robot raven_2, 18 links, 17 joints
Links:
- link 0_link: geometry collision box size=0.01 0.01 0.01; visual box size=0.01 0.01 0.01

Commit message: Changes made for trajopt working

File: raven_visualization/ravenII_2arm.urdf (robot description, URDF)
Before this commit: robot raven_2, 17 links, 16 joints
Links:
- added link grasper3_L; visual mesh filename=package://raven_visualization/Raven_files/dome.dae
Joints:
- added joint grasper_joint_3_L: type revolute, parent wrist_L, child grasper3_L, origin xyz=0.00680 0.00904 -0.00452 rpy=0 0 0, axis 0.5648    -0.1427   0.8128, limit lower=-2 upper=2 effort=1000.0 velocity=.5

Commit message: transparent dome in rviz when aplha set to 0.5

File: raven_visualization/ravenII_2arm.urdf (robot description, URDF)
Before this commit: robot raven_2, 18 links, 17 joints
Links:
- removed link grasper3_L
- added link dome; visual mesh filename=package://raven_visualization/Raven_files/dome.dae
Joints:
- removed joint grasper_joint_3_L
- added joint dome: type fixed, parent 0_link, child dome, origin xyz=0.00680 0.00904 -0.00452 rpy=0 0 0, axis 0    0   0, limit lower=-2 upper=2 effort=1000.0 velocity=.5

Commit message: added gazebo simulation

File: raven_visualization/ravenII_2arm.urdf (robot description, URDF)
Before this commit: robot raven_2, 17 links, 16 joints
Links:
- added link wood_R, mass 1; collision mesh filename=/home/homa/Downloads/Ring.dae; visual mesh filename=/home/homa/Downloads/Ring.dae
- added link world
- link 0_link: mass None -> 1; geometry visual box size=0.01 0.01 0.01
- link base_link_L: mass None -> 10; geometry visual box size=0.43 0.25 0.32
- link base_link_R: mass None -> 10; geometry visual box size=0.43 0.25 0.32
- link grasper1_L: mass None -> 1; geometry collision mesh filename=package://raven_visualization/Raven_files/left_arm/grasper_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; visual mesh filename=package://raven_visualization/Raven_files/left_arm/grasper_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
- link grasper1_R: mass None -> 1; geometry collision mesh filename=package://raven_visualization/Raven_files/right_arm/grasper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; visual mesh filename=package://raven_visualization/Raven_files/right_arm/grasper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
- link grasper2_L: mass None -> 1; geometry collision mesh filename=package://raven_visualization/Raven_files/left_arm/grasper_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; visual mesh filename=package://raven_visualization/Raven_files/left_arm/grasper_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
- link grasper2_R: mass None -> 1; geometry collision mesh filename=package://raven_visualization/Raven_files/right_arm/grasper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; visual mesh filename=package://raven_visualization/Raven_files/right_arm/grasper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
- link instrument_shaft_L: mass None -> 1; geometry collision mesh filename=package://raven_visualization/Raven_files/left_arm/instrume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; visual mesh filename=package://raven_visualization/Raven_files/left_arm/instrume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
- link instrument_shaft_R: mass None -> 10; geometry collision mesh filename=package://raven_visualization/Raven_files/right_arm/instrum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; visual mesh filename=package://raven_visualization/Raven_files/right_arm/instrum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
- link link1_L: mass None -> 10; geometry collision mesh filename=package://raven_visualization/Raven_files/left_arm/link1_w_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; visual mesh filename=package://raven_visualization/Raven_files/left_arm/link1_w_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
- link link1_R: mass None -> 10; geometry collision mesh filename=package://raven_visualization/Raven_files/right_arm/link1_w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; visual mesh filename=package://raven_visualization/Raven_files/right_arm/link1_w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
- link link2_L: mass None -> 10; geometry collision mesh filename=package://raven_visualization/Raven_files/left_arm/link2.dae; visual mesh filename=package://raven_visualization/Raven_files/left_arm/link2.dae
- link link2_R: mass None -> 10; geometry collision mesh filename=package://raven_visualization/Raven_files/right_arm/link2.d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; visual mesh filename=package://raven_visualization/Raven_files/right_arm/link2.d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
- link link3_L: mass None -> 10; geometry collision mesh filename=package://raven_visualization/Raven_files/left_arm/link3.dae; visual mesh filename=package://raven_visualization/Raven_files/left_arm/link3.dae
- link link3_R: mass None -> 10; geometry collision mesh filename=package://raven_visualization/Raven_files/right_arm/link3.d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; visual mesh filename=package://raven_visualization/Raven_files/right_arm/link3.d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
- link wrist_L: mass None -> 1; geometry collision mesh filename=package://raven_visualization/Raven_files/left_arm/wrist.dae; visual mesh filename=package://raven_visualization/Raven_files/left_arm/wrist.dae
- link wrist_R: mass None -> 1; geometry collision mesh filename=package://raven_visualization/Raven_files/right_arm/wrist.d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; visual mesh filename=package://raven_visualization/Raven_files/right_arm/wrist.d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
Joints:
- added joint fixed: type fixed, parent world, child 0_link
- added joint pegW: type fixed, parent wrist_R, child wood_R, origin xyz=-2.00680 -0.0104 -1.00452 rpy=0 0 0, axis 0.5648    0.1427   0.8128, limit lower=-2 upper=2 effort=1000.0 velocity=.5

Commit message: Decreased the mass of links in ravenII_2arm.urdf

File: raven_visualization/ravenII_2arm.urdf (robot description, URDF)
Before this commit: robot raven_2, 19 links, 18 joints
Links:
- link base_link_L: mass 10 -> 1
- link base_link_R: mass 10 -> 1
- link instrument_shaft_R: mass 10 -> 1
- link link1_L: mass 10 -> 1
- link link1_R: mass 10 -> 1
- link link2_L: mass 10 -> 1
- link link2_R: mass 10 -> 1
- link link3_L: mass 10 -> 1
- link link3_R: mass 10 -> 1
