Commit message: Pushing latest changes from Parisa (robot goes through box)

File: raven_visualization/box.urdf (robot description, URDF)
Before this commit: robot box_Demo, 1 links, 0 joints
Links:
- link box: mass 10 -> 1000

File: raven_visualization/ravenII_2arm.urdf (robot description, URDF)
Before this commit: robot raven_2, 19 links, 18 joints
Links:
- removed link wood_R
- link base_link_L: mass 1 -> 10
- link base_link_R: mass 1 -> 10
- link instrument_shaft_R: mass 1 -> 10
- link link1_L: mass 1 -> 10
- link link1_R: mass 1 -> 10
- link link2_L: mass 1 -> 10
- link link2_R: mass 1 -> 10
- link link3_L: mass 1 -> 10
- link link3_R: mass 1 -> 10
Joints:
- removed joint pegW

Commit message: Gazebo running with changes in the urdf

File: raven_visualization/box.urdf (robot description, URDF)
Before this commit: robot box_Demo, 1 links, 0 joints
Links:
- link box: mass 1000 -> 10

File: raven_visualization/ravenII_2arm.urdf (robot description, URDF)
Before this commit: robot raven_2, 18 links, 17 joints
Links:
- link 0_link: mass 1 -> None; geometry visual box size=0.00001 0.00001 0.00001
- link base_link_L: geometry visual mesh filename=package://raven_visualization/Raven_files/left_arm/base_w_m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
- link base_link_R: geometry visual mesh filename=package://raven_visualization/Raven_files/right_arm/base_w_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
- link instrument_shaft_L: mass 1 -> 10

Commit message: Changed made while testing dyn_sim + gui

File: raven_visualization/box.urdf (robot description, URDF)
Before this commit: robot box_Demo, 1 links, 0 joints
Links:
- link box: mass 10 -> 1
