Commit message: gazebo simulator works with video recording

File: raven_visualization/ravenII_2arm_correct.urdf (robot description, URDF)
Before this commit: robot raven_2, 18 links, 17 joints
Links:
- link 0_link: mass 1 -> None; geometry visual box size=0.00001 0.00001 0.00001
- link base_link_L: geometry visual mesh filename=package://raven_visualization/Raven_files/left_arm/base_w_m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
- link base_link_R: geometry visual mesh filename=package://raven_visualization/Raven_files/right_arm/base_w_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
- link instrument_shaft_L: mass 1 -> 10
